Commit message: easier parameter

File: envs/cyl.urdf (robot description, URDF)
Before this commit: robot paddle, 1 links, 0 joints
Links:
- link paddleLink: mass 30.0 -> 3.0

Commit message: turned on gravity haha. Then adjusted other parameters accordingly

File: envs/cyl.urdf (robot description, URDF)
Before this commit: robot paddle, 1 links, 0 joints
Links:
- link paddleLink: mass 3.0 -> 1.0

Commit message: Refactor to use transition model functions

File: envs/cyl.urdf (robot description, URDF)
Before this commit: robot paddle, 1 links, 0 joints
Links:
- link paddleLink: mass 1.0 -> 0.5

Commit message: simulation should be substantially faster

File: envs/cyl.urdf (robot description, URDF)
Before this commit: robot paddle, 1 links, 0 joints
Links:
- link paddleLink: mass 0.5 -> 0.1

Commit message: Smoother simulation viewing when gui is turned on

File: envs/cyl.urdf (robot description, URDF)
Before this commit: robot paddle, 1 links, 0 joints
Links:
- link paddleLink: mass 0.1 -> 0.5
