Commit message: pass the example

File: envs/paddle.urdf (robot description, URDF)
Before this commit: robot paddle, 4 links, 3 joints
Links:
- link paddleLink: geometry collision box size=0.8 0.1 0.2

Commit message: got rid of joint limits

File: envs/paddle.urdf (robot description, URDF)
Before this commit: robot paddle, 4 links, 3 joints
Joints:
- joint inter1_to_2: limit lower=-1 upper=1 effort=1.0 velocity=1.5 -> lower=-6.28 upper=6.28 effort=1.0 velocity=1.5
- joint prism_base_to_inter1: limit lower=-1 upper=1 effort=10.0 velocity=3.5 -> lower=-6.28 upper=6.28 effort=10.0 velocity=3.5
- joint revolute_inter2_to_paddle: limit lower=-3. upper=3. effort=100.0 velocity=30.5 -> lower=-6.28 upper=6.28 effort=100.0 velocity=30.5

Commit message: added some debug code, runs and looks OK. prints out large errors sometimes

File: envs/paddle.urdf (robot description, URDF)
Before this commit: robot paddle, 4 links, 3 joints
Joints:
- joint prism_base_to_inter1: limit lower=-6.28 upper=6.28 effort=10.0 velocity=3.5 -> lower=-6.28 upper=6.28 effort=1.0 velocity=3.5
- joint revolute_inter2_to_paddle: limit lower=-6.28 upper=6.28 effort=100.0 velocity=30.5 -> lower=-6.28 upper=6.28 effort=1.0 velocity=30.5

Commit message: consistent physics that are followed

File: envs/paddle.urdf (robot description, URDF)
Before this commit: robot paddle, 4 links, 3 joints
Links:
- link paddleLink: mass 1.0 -> 0.3
Joints:
- joint inter1_to_2: limit lower=-6.28 upper=6.28 effort=1.0 velocity=1.5 -> lower=-156.28 upper=156.28 effort=0.1 velocity=30.5
- joint prism_base_to_inter1: limit lower=-6.28 upper=6.28 effort=1.0 velocity=3.5 -> lower=-156.28 upper=156.28 effort=0.1 velocity=30.5
- joint revolute_inter2_to_paddle: limit lower=-6.28 upper=6.28 effort=1.0 velocity=30.5 -> lower=-16.28 upper=16.28 effort=5.0 velocity=30.5
